File: lib/blocks/xiao-reversible-block.kicad_blocks/xiao-reversible-block.kicad_block/xiao-reversible-block.kicad_sch (KiCad schematic)
At the start: 34 parts, among them J1 Conn_01x02, U1 XIAO-nRF52840-DIP

Commit message: refactor: bugfixes, refinements
- fix netnames: no _L/_R suffix required, same nets
- added traces to through holes
- fixed orientation of 0R resistors
- ungrouped 0R resistors (too difficult to access)
Connections:
- net P0.03_A1_D1_L is gone; now on net P0.03_A1_D1: RL2.1
- net P0.03_A1_D1_R is gone; now on net GND: RL13.2
- net P0.28_A2_D2_L is gone; now on net P0.28_A2_D2: RL3.1
- net P0.28_A2_D2_R is gone; now on net 3V3: RL12.2
- net P1.12_D7_RX_L is gone; now on net P1.11_D6_TX: RR8.1
- net P1.12_D7_RX_R is gone; now on net P1.12_D7_RX: RR7.2
- net P1.13_D8_SCK_L is gone; now on net P0.05_A5_D5_SCL: RR9.1
- net P1.13_D8_SCK_R is gone; now on net P1.13_D8_SCK: RR6.2
- net P1.14_D9_MISO_L is gone; now on net P0.04_A4_D4_SDL: RR10.1
- net P1.14_D9_MISO_R is gone; now on net P1.14_D9_MISO: RR5.2
- net P1.15_D10_MOSI_L is gone; now on net P0.29_A3_D3: RR11.1
- net P1.15_D10_MOSI_R is gone; now on net P1.15_D10_MOSI: RR4.2
- net VBUS_L is gone; now on net P.0.02_A0_D0: RR14.1
- net VBUS_R is gone; now on net VBUS: RR1.2
- net BAT+: now also RBR2.1; no longer RBL2.2
- net BAT-: now also RBL2.2; no longer RBR2.1
- net 3V3_L renamed P0.28_A2_D2
- net 3V3_R renamed 3V3
- net GND_L renamed P0.03_A1_D1
- net GND_R renamed GND
- net P.0.02_A0_D0_L renamed P.0.02_A0_D0
- net P.0.02_A0_D0_R renamed VBUS
- net P0.04_A4_D4_SDL_L renamed P0.04_A4_D4_SDL
- net P0.04_A4_D4_SDL_R renamed P1.14_D9_MISO
- net P0.05_A5_D5_SCL_L renamed P0.05_A5_D5_SCL
- net P0.05_A5_D5_SCL_R renamed P1.13_D8_SCK
- net P0.29_A3_D3_L renamed P0.29_A3_D3
- net P0.29_A3_D3_R renamed P1.15_D10_MOSI
- net P1.11_D6_TX_L renamed P1.11_D6_TX
- net P1.11_D6_TX_R renamed P1.12_D7_RX
