File: lib/blocks/xiao-reversible-block.kicad_blocks/xiao-reversible-block.kicad_block/xiao-reversible-block.kicad_pcb (KiCad board)
At the start: 2 copper layers, 34 parts, among them J1 Conn_01x02, U1 XIAO-nRF52840-DIP

Commit message: fix: fix bugs and improve
- typo: SDL -> SDA
- replaced GND net by actual ground symbol
- fixed power flags for ERC
Connections:
- net /3V3 renamed +3V3
- net /BAT+ renamed BAT+
- net /P0.04_A4_D4_SDL renamed /P0.04_A4_D4_SDA
- net /VBUS renamed +5V
- RBL2 pad 2: /BAT- -> GND
- RBR1 pad 2: /BAT- -> GND
- RL13 pad 2: /GND -> GND
- RR2 pad 2: /GND -> GND
Routing:
- net BAT+: track 0.00 -> 12.9 mm, vias 0 -> 1
