File: lib/blocks/xiao-reversible-block.kicad_blocks/xiao-reversible-block.kicad_block/xiao-reversible-block.kicad_pcb (KiCad board)
At the start: 2 copper layers, 34 parts, among them J1 Conn_01x02, U1 XIAO-nRF52840-DIP

Commit message: fix: decrease header spacing, remove JST battery connector
Parts:
- removed J1: Conn_01x02, Connector_JST:JST_PH_S2B-PH-K_1x02_P2.00mm_Horizontal
- removed RBL1, RBL2, RBR1, RBR2: 0R, xiao-reversible-block:R_0603_1608Metric_Pad0.98x0.95mm_HandSolder_0R
- moved RL1 0.13 mm to (153.6, 80.2)
- moved RR1 0.13 mm to (153.6, 80.2)
- moved RL10 0.12 mm to (159.6, 90.3)
- moved RL12 0.12 mm to (159.6, 85.3)
- moved RL14 0.12 mm to (159.6, 80.2)
- moved RL5 0.12 mm to (153.6, 90.3)
- moved RL6 0.12 mm to (153.6, 92.9)
- moved RL7 0.12 mm to (153.6, 95.4)
- moved RL8 0.12 mm to (159.6, 95.4)
- moved RL9 0.12 mm to (159.6, 92.9)
- moved RR10 0.12 mm to (159.6, 90.3)
- moved RR12 0.12 mm to (159.6, 85.3)
- moved RR14 0.12 mm to (159.6, 80.2)
- moved RR5 0.12 mm to (153.6, 90.3)
- moved RR6 0.12 mm to (153.6, 92.9)
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Routing:
- net BAT+: track 12.9 -> 0.00 mm, vias 1 -> 0
- net Net-(J1-Pin_1): track 5.39 -> 0.00 mm
- net Net-(J1-Pin_2): track 5.39 -> 0.00 mm
- net Net-(U1-P0.29_A3_D3): track 8.31 -> 7.81 mm
- net Net-(U1-P0.28_A2_D2): track 8.31 -> 7.81 mm
- net Net-(U1-P0.03_A1_D1): track 8.31 -> 7.81 mm
- net Net-(U1-P0.02_A0_D0): track 8.31 -> 7.81 mm
